File: chainable-batmon.kicad_pcb (KiCad board)
At the start: 2 copper layers, 38 x 30 mm, 19 parts, among them J1 TRS-jack, J2 TRS-jack, J3 Bat, U1 MCP1700-5002E_SOT23, U2 LM393, U3 SFH617A-1

Commit message: Added renders and updated readme
Parts:
- added G***: LOGO, graphics:kiwi, B.Cu at (107.2, 104.5)
Other:
- board text added: "git.io/batmon"
- board text added: "v1.0.0"
Changed lines of the file:
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@@
   (general
     (thickness 1.6)
-    (drawings 14)
+    (drawings 16)
     (tracks 96)
     (zones 0)
-    (modules 19)
+    (modules 20)
     (nets 13)
   )
@@
   )
   (setup
-    (last_trace_width 0.4)
+    (last_trace_width 0.2)
     (user_trace_width 0.4)
     (user_trace_width 0.6)
@@
     (pad_to_mask_clearance 0.2)
     (aux_axis_origin 0 0)
-    (visible_elements FFFFFF7F)
+    (visible_elements 7FFFFFFF)
     (pcbplotparams
       (layerselection 0x010fc_ffffffff)
@@
     (pad 1 np_thru_hole circle (at 0 0) (size 3.2 3.2) (drill 3.2) (layers *.Cu *.Mask))
   )
+  (module graphics:kiwi (layer B.Cu)
+    (at 107.25 104.5 180)
+    (fp_text reference G*** (at 0 0 180) (layer B.SilkS) hide
+      (effects (font (size 1.524 1.524) (thickness 0.3)) (justify mirror))
+    )
+    (fp_text value LOGO (at 0.75 0 180) (layer B.SilkS) hide
+      (effects (font (size 1.524 1.524) (thickness 0.3)) (justify mirror))
+    )
+    (fp_poly (pts (xy -3.693852 2.064291) (xy -3.542325 1.914383) (xy -3.504409 1.813591) (xy -3.509965 1.575994)
+      (xy -3.630403 1.41603) (xy -3.819581 1.358933) (xy -4.03136 1.429937) (xy -4.100286 1.487715)
+      (xy -4.212314 1.631567) (xy -4.205969 1.764741) (xy -4.079911 1.94871) (xy -3.890351 2.079796)
+      (xy -3.693852 2.064291)) (layer B.Mask) (width 0.01))
+    (fp_poly (pts (xy -4.818523 2.053158) (xy -4.667994 1.909407) (xy -4.577302 1.755582) (xy -4.572 1.720956)
+      (xy -4.63549 1.59377) (xy -4.778999 1.452948) (xy -4.932091 1.362543) (xy -4.974786 1.354667)
+      (xy -5.10451 1.40929) (xy -5.200953 1.487715) (xy -5.308906 1.643614) (xy -5.334 1.735667)
+      (xy -5.268279 1.899506) (xy -5.119133 2.050966) (xy -4.960075 2.116667) (xy -4.818523 2.053158)) (layer B.Mask) (width 0.01))
+    (fp_poly (pts (xy 2.887919 4.58736) (xy 3.833817 4.274527) (xy 4.117897 4.149723) (xy 4.761726 3.786098)
+      (xy 5.263271 3.352963) (xy 5.641455 2.832624) (xy 5.749105 2.624667) (xy 5.842579 2.412133)
+      (xy 5.905184 2.216286) (xy 5.942999 1.994992) (xy 5.962106 1.706112) (xy 5.968583 1.307512)
+      (xy 5.969 1.100667) (xy 5.956755 0.509509) (xy 5.909333 0.024578) (xy 5.810705 -0.385255)
+      (xy 5.644844 -0.751121) (xy 5.395719 -1.10415) (xy 5.047301 -1.475471) (xy 4.583563 -1.896215)
+      (xy 4.302718 -2.135456) (xy 4.02436 -2.401906) (xy 3.783992 -2.688996) (xy 3.64937 -2.90302)
+      (xy 3.523194 -3.251007) (xy 3.476915 -3.580932) (xy 3.512718 -3.846732) (xy 3.598333 -3.979333)
+      (xy 3.714614 -4.117107) (xy 3.670273 -4.202538) (xy 3.466241 -4.234024) (xy 3.450167 -4.23416)
+      (xy 3.217125 -4.270896) (xy 2.917622 -4.364176) (xy 2.7305 -4.441932) (xy 2.286 -4.648876)
+      (xy 2.286 -4.429447) (xy 2.277846 -4.305307) (xy 2.225923 -4.246079) (xy 2.089037 -4.237194)
+      (xy 1.825998 -4.264083) (xy 1.820333 -4.264749) (xy 1.514506 -4.282497) (xy 1.361604 -4.250446)
+      (xy 1.355241 -4.176196) (xy 1.489036 -4.067347) (xy 1.756602 -3.931499) (xy 2.151557 -3.776252)
+      (xy 2.263331 -3.737379) (xy 2.921 -3.513666) (xy 2.946269 -2.982089) (xy 2.953571 -2.68129)
+      (xy 2.927955 -2.488641) (xy 2.851626 -2.343637) (xy 2.714247 -2.193221) (xy 2.446932 -2.002804)
+      (xy 2.19954 -1.970999) (xy 1.984188 -2.087266) (xy 1.812992 -2.341062) (xy 1.698071 -2.721848)
+      (xy 1.654605 -3.115035) (xy 1.6332 -3.598333) (xy 1.308198 -3.651171) (xy 0.962159 -3.785425)
+      (xy 0.788352 -3.947504) (xy 0.593508 -4.191) (xy 0.593087 -3.910127) (xy 0.579886 -3.722971)
+      (xy 0.518368 -3.664741) (xy 0.402167 -3.687025) (xy 0.197207 -3.787971) (xy 0.021167 -3.919156)
+      (xy -0.169333 -4.093517) (xy -0.169333 -3.915921) (xy -0.092981 -3.666871) (xy 0.108837 -3.425469)
+      (xy 0.395265 -3.231145) (xy 0.632423 -3.142147) (xy 0.814137 -3.093428) (xy 0.935376 -3.034764)
+      (xy 1.015647 -2.932372) (xy 1.07446 -2.752469) (xy 1.131324 -2.461271) (xy 1.175594 -2.201541)
+      (xy 1.212082 -1.886404) (xy 1.192707 -1.711178) (xy 1.171301 -1.68466) (xy 1.06511 -1.6545)
+      (xy 0.819487 -1.601391) (xy 0.46194 -1.530762) (xy 0.019976 -1.448042) (xy -0.478898 -1.35866)
+      (xy -0.493117 -1.356167) (xy -1.435837 -1.181097) (xy -2.227053 -1.011267) (xy -2.884263 -0.841284)
+      (xy -3.424961 -0.665755) (xy -3.866645 -0.479289) (xy -4.22681 -0.276494) (xy -4.402667 -0.151269)
+      (xy -4.598961 0.044831) (xy -4.787785 0.303076) (xy -4.932019 0.564894) (xy -4.99454 0.771715)
+      (xy -4.9949 0.783167) (xy -5.056784 0.901362) (xy -5.215467 0.931334) (xy -5.446367 1.004309)
+      (xy -5.713063 1.20913) (xy -5.734037 1.22977) (xy -5.909949 1.420236) (xy -5.991494 1.578368)
+      (xy -6.004413 1.769976) (xy -5.897187 1.769976) (xy -5.796292 1.466808) (xy -5.610837 1.227233)
+      (xy -5.369574 1.073315) (xy -5.101252 1.027117) (xy -4.834623 1.110705) (xy -4.707659 1.211311)
+      (xy -4.552999 1.38592) (xy -4.457508 1.528811) (xy -4.402415 1.608665) (xy -4.347826 1.528811)
+      (xy -4.170052 1.278897) (xy -3.918274 1.092203) (xy -3.656995 1.016081) (xy -3.649237 1.016)
+      (xy -3.343607 1.087415) (xy -3.111692 1.276258) (xy -2.960248 1.544425) (xy -2.896026 1.853814)
+      (xy -2.92578 2.166321) (xy -3.056263 2.443845) (xy -3.294229 2.648281) (xy -3.354869 2.676859)
+      (xy -3.67612 2.742478) (xy -3.965173 2.649251) (xy -4.233704 2.398157) (xy -4.375884 2.255616)
+      (xy -4.457015 2.251147) (xy -4.463167 2.263701) (xy -4.63797 2.530318) (xy -4.909691 2.717244)
+      (xy -5.043423 2.758913) (xy -5.3137 2.733042) (xy -5.578915 2.582122) (xy -5.789138 2.344387)
+      (xy -5.884772 2.114672) (xy -5.897187 1.769976) (xy -6.004413 1.769976) (xy -6.005088 1.779973)
+      (xy -5.990448 1.965575) (xy -5.93991 2.267824) (xy -5.836931 2.477868) (xy -5.682209 2.640805)
+      (xy -5.452173 2.787857) (xy -5.191512 2.871675) (xy -4.954943 2.882931) (xy -4.797185 2.812292)
+      (xy -4.783677 2.794018) (xy -4.693683 2.792826) (xy -4.518465 2.888708) (xy -4.389159 2.984518)
+      (xy -4.242416 3.098042) (xy -4.110832 3.1764) (xy -3.958119 3.2277) (xy -3.747985 3.260053)
+      (xy -3.44414 3.281568) (xy -3.010294 3.300355) (xy -2.968435 3.302) (xy -1.889913 3.344334)
+      (xy -1.43179 3.694711) (xy -0.642518 4.199174) (xy 0.190098 4.541164) (xy 1.060049 4.720186)
+      (xy 1.961326 4.735749) (xy 2.887919 4.58736)) (layer B.Mask) (width 0.01))
+  )
+  (gr_text v1.0.0 (at 105.5 111.25) (layer F.SilkS)
+    (effects (font (size 1.25 1.25) (thickness 0.2)))
+  )
+  (gr_text git.io/batmon (at 96.75 99.25 270) (layer F.SilkS)
+    (effects (font (size 1.25 1.25) (thickness 0.2)))
+  )
   (gr_text bat (at 131 106.75 90) (layer F.SilkS)
